File: minisumo_2025.kicad_pcb (KiCad board)
At the start: 4 copper layers, 40.1 x 90 mm, 117 parts, among them J1 USB_C Connector, J10 DISTANCE_R90, J11 DISTANCE_R, J12 DISTANCE_RF, J13 DISTANCE_L90, J14 DISTANCE_L, J15 LINE_LEFT, J16 DISTANCE_LF, J2 SERVO, J3 START_MODULE, J4 MOTOR1, J5 MOTOR2, J6 BATT_IN, J8 DISTANCE_CENTER, J9 LINE_RIGHT, SW1 RESET, SW2 CASE, SW5 BOOT, U1 LMR33630ADDAR, U2 USBLC6-2P6, U3 ESP32-S3-WROOM-1, U4 TLV75730PDBVR, U5 TXS0108ERGYR, U6 MC33926PNB, U7 MC33926PNB

Commit message: saved required changes
Parts:
- removed C33: 0.1uF, Capacitor_SMD:C_0402_1005Metric
- added C30: 0.1uF, Capacitor_SMD:C_0402_1005Metric, F.Cu at (139.3, 108.6)
- U5: value TXS0108ERGYR -> TXS0108EPWR; footprint footprints:DQS20_TEX -> footprints:SOP65P640X120-20N
- moved C29 5.06 mm to (148.6, 108.9), turned to -90 degrees
- moved U5 2.37 mm to (144.2, 106.2)
- moved D3 0.35 mm to (127.9, 128.5)
Connections:
- J1 pad S1: GND -> unconnected-(J1-SHIELD-PadS1)_1
- R22 pad 1: GND -> unconnected-(R22-Pad1)
- U3 pad 4: /DISTANCE_R90 -> /DISTANCE_L90
- U3 pad 5: /DISTANCE_R -> /DISTANCE_L
- U3 pad 6: /DISTANCE_RF -> /DISTANCE_LF
- U3 pad 7: /DISTANCE_LF -> /DISTANCE_RF
- U3 pad 8: /DISTANCE_L -> /DISTANCE_R
- U3 pad 9: /DISTANCE_L90 -> /DISTANCE_R90
- U5 pad 10: unconnected-(U5-A8-Pad10) -> +3V3
- U5 pad 11: unconnected-(U5-B8-Pad11) -> GND
- U5 pad 12: /DISTANCE_R90_OUT -> unconnected-(U5-B8-Pad12)
- U5 pad 13: /DISTANCE_R_OUT -> /DISTANCE_R90_OUT
- U5 pad 14: /DISTANCE_RF_OUT -> /DISTANCE_R_OUT
- U5 pad 15: GND -> /DISTANCE_RF_OUT
- U5 pad 16: +5V -> unconnected-(U5-B4-Pad16)
- U5 pad 17: unconnected-(U5-B4-Pad17) -> /DISTANCE_LF_OUT
- U5 pad 18: /DISTANCE_LF_OUT -> /DISTANCE_L_OUT
- U5 pad 19: /DISTANCE_L_OUT -> +5V
- U5 pad 2: /DISTANCE_L -> +3V3
- U5 pad 3: /DISTANCE_LF -> /DISTANCE_L
- U5 pad 4: unconnected-(U5-A4-Pad4) -> /DISTANCE_LF
- U5 pad 5: +3V3 -> unconnected-(U5-A4-Pad5)
- U5 pad 6: +3V3 -> /DISTANCE_RF
- U5 pad 7: /DISTANCE_RF -> /DISTANCE_R
- U5 pad 8: /DISTANCE_R -> /DISTANCE_R90
- U5 pad 9: /DISTANCE_R90 -> unconnected-(U5-A8-Pad9)
Routing:
- net /DISTANCE_L90: track 17.5 -> 10.0 mm
- net +3V3: track 301.2 -> 307.6 mm
- net /DISTANCE_L: track 17.4 -> 12.4 mm
- net /DISTANCE_RF: track 20.4 -> 15.8 mm
- net GND: track 26.5 -> 22.7 mm, vias 151 -> 216
- net +5V: track 17.6 -> 21.1 mm, vias 25 -> 28
- net /DISTANCE_LF: track 17.1 -> 13.7 mm
- net /DISTANCE_R: track 20.2 -> 16.9 mm
- net /DISTANCE_R90: track 19.8 -> 18.1 mm
- net /DISTANCE_RF_OUT: track 38.0 -> 39.0 mm
- net /DISTANCE_R_OUT: track 41.9 -> 42.7 mm
- net /DISTANCE_R90_OUT: track 49.1 -> 49.7 mm
Other:
- board text added: "PULLDOWN"
- board text added: "PULLUP"
- board text removed: "4"

Commit message: more
Other:
- board text added: "- dimensiuni componente mai mari de 0603 - thermal relief-uri pe ground - condensatori de mai multe valori pe batt input - valori VOLTAGE condensatori x3 mai mari - piese corecte - spatiere mai mare intre componente - D1 - low, D2 - high, SLEW - floating, INV - floating, FB - rezistenta la GND - pad-urile de breakout sa fie la 3v3, fara rezistente - leduri mai putin puternice pt battery indicator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"
- board text added: "PROBLEME"
Changed lines of the file:
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@@
 		(layer "Edge.Cuts")
+	)
+	(gr_text "PROBLEME"
+		(at 173.5 51.5 0)
+		(layer "F.Cu")
+		(effects
+			(font
+				(size 1.5 1.5)
+				(thickness 0.3)
+				(bold yes)
+			)
+			(justify left bottom)
+		)
+	)
+	(gr_text "- dimensiuni componente mai mari de 0603\n- thermal relief-uri pe ground\n- condensatori de mai multe valori pe batt input\n- valori VOLTAGE condensatori x3 mai mari\n- piese corecte\n- spatiere mai mare intre componente\n- D1 - low, D2 - high, SLEW - floating, INV - floating, FB - rezistenta la GND\n- pad-urile de breakout sa fie la 3v3, fara rezistente\n- leduri mai putin puternice pt battery indicator, poate de culori diferite (verde)\n- led indicator conectat la esp\n- regulator de 3v3 nu de 3v\n- verificare silkscreen (nume, plasament)\n- numele pentru pad-uri sa fie puse deasupra\n- breakout pentru 3V3 si 5V\n- decupat colturi roti"
+		(at 173 91 0)
+		(layer "F.Cu")
+		(effects
+			(font
+				(size 1.5 1.5)
+				(thickness 0.1875)
+			)
+			(justify left bottom)
+		)
 	)
 	(gr_text "IO21"

Commit message: test board layout
Parts:
- removed ?: , 
- removed C1, C12, C16, C18, C25, C26, C29, C3, C30, C6, C7: 0.1uF, Capacitor_SMD:C_0402_1005Metric
- removed C10, C8, C9: 47uF, Capacitor_SMD:C_1210_3225Metric
- removed C11, C21 (x5), C23, C27, C28: 100nF, Capacitor_SMD:C_0603_1608Metric
- removed C13: 1uF, Capacitor_SMD:C_0603_1608Metric
- removed C14, C15, C17, C4: 10uF, Capacitor_SMD:C_1210_3225Metric
- removed C19, C20: 33nF, Capacitor_SMD:C_0603_1608Metric
- removed C2: 10uF, Capacitor_SMD:C_0603_1608Metric
- removed C32: 1uF, Capacitor_SMD:C_0402_1005Metric
- removed C5: 220nF, Capacitor_SMD:C_0805_2012Metric
- removed D2, D7, D8, D9: 2Vf, 20mA, RED, LED_SMD:LED_0603_1608Metric
- removed D3: D_Schottky_Small, Diode_SMD:D_SOD-123
- removed D4: 10V, Diode_SMD:Nexperia_CFP3_SOD-123W
- removed D5: 8.2V, Diode_SMD:Nexperia_CFP3_SOD-123W
- removed D6: 6V, Diode_SMD:Nexperia_CFP3_SOD-123W
- removed J2: SERVO, Connector_JST:JST_XH_B3B-XH-A_1x03_P2.50mm_Vertical
- removed JP1, JP2, JP3, JP4, JP5, JP6, JP7, JP8: SolderJumper_3_Open, Jumper:SolderJumper-3_P1.3mm_Open_RoundedPad1.0x1.5mm_NumberLabels
- removed R1, R13, R15, R7: 10k, Resistor_SMD:R_0402_1005Metric
- removed R10, R11, R12, R14, R16, R19, R20, R9: 1k, Resistor_SMD:R_0402_1005Metric
- removed R17: 412, Resistor_SMD:R_0402_1005Metric
- removed R18: 300, Resistor_SMD:R_0402_1005Metric
- removed R2, R3: 5k1, Resistor_SMD:R_0402_1005Metric
- removed R21, R23: 2k, Resistor_SMD:R_0402_1005Metric
- removed R22, R24: 3.3k, Resistor_SMD:R_0402_1005Metric
- removed R25: 200, Resistor_SMD:R_0402_1005Metric
- removed R4: 100k, Resistor_SMD:R_0402_1005Metric
- removed R5: 22.1k, Resistor_SMD:R_0402_1005Metric
- removed R6: 68, Resistor_SMD:R_0402_1005Metric
- removed R8: 5k, Resistor_SMD:R_0402_1005Metric
- removed TP1: GPIO13, TestPoint:TestPoint_Pad_1.5x1.5mm
- removed TP10: SLEW_2, TestPoint:TestPoint_Pad_1.5x1.5mm
- removed TP11: INV_2, TestPoint:TestPoint_Pad_1.5x1.5mm
- removed TP12: D1_2, TestPoint:TestPoint_Pad_1.5x1.5mm
- removed TP13: D2_2, TestPoint:TestPoint_Pad_1.5x1.5mm
- removed TP2: GPIO47, TestPoint:TestPoint_Pad_1.5x1.5mm
- removed TP3: GPIO48, TestPoint:TestPoint_Pad_1.5x1.5mm
- removed TP4: GPIO21, TestPoint:TestPoint_Pad_1.5x1.5mm
- removed TP5: GPIO14, TestPoint:TestPoint_Pad_1.5x1.5mm
- removed TP6: SLEW_1, TestPoint:TestPoint_Pad_1.5x1.5mm
- removed TP7: INV_1, TestPoint:TestPoint_Pad_1.5x1.5mm
- removed TP8: D1_1, TestPoint:TestPoint_Pad_1.5x1.5mm
- removed TP9: D2_1, TestPoint:TestPoint_Pad_1.5x1.5mm
- added C31: 4.7uF, Capacitor_SMD:C_1210_3225Metric, F.Cu at (128.4, 102.4)
- added C33: 10uF, Capacitor_THT:C_Radial_D6.3mm_H11.0mm_P2.50mm, F.Cu at (127.3, 84.8)
- J1, J10, J11, J12, J13, J14, J15, J16, J8, J9, U2: moved to F.Cu
- J4, J5: moved to B.Cu
- U3: footprint RF_Module:ESP32-S3-WROOM-1 -> RF_Module:ESP32-S3-WROOM-1U; moved to F.Cu
- U4: value TLV75730PDBVR -> TLV75733PDBVR
- moved SW2 71.4 mm to (146.4, 70.4), turned to 0 degrees
- moved SW1 70.0 mm to (152.8, 70.4), turned to 0 degrees
- moved J1 69.2 mm to (166.8, 74.0), turned to 90 degrees
- moved SW5 67.4 mm to (140.0, 70.4), turned to 0 degrees
- moved U3 58.7 mm to (123.6, 54.8), turned to 0 degrees
- moved U2 58.3 mm to (160.3, 73.8), turned to 0 degrees
- moved C24 53.5 mm to (145.6, 106.0), turned to 0 degrees
- moved D1 44.8 mm to (127.0, 130.8), turned to 0 degrees
- moved U6 37.4 mm to (138.0, 108.0)
- moved J5 37.3 mm to (137.4, 96.4), turned to -90 degrees
- moved U5 36.3 mm to (129.7, 72.9), turned to -90 degrees
- moved L1 32.7 mm to (112.4, 128.6), turned to 0 degrees
- moved J8 26.4 mm to (127.2, 115.6)
- moved U1 24.3 mm to (123.3, 125.1), turned to 0 degrees
- moved C22 23.3 mm to (145.1, 78.0), turned to 0 degrees
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Connections:
- U1 pad V: GND -> (no net)
- U6 pad 1: /GPIO35 -> /GPIO17
- U6 pad 16: /ND2_1 -> +3V3
- U6 pad 2: /GPIO36 -> /GPIO21
- U6 pad 26: /D1_1 -> GND
- U6 pad 8: unconnected-(U6-FB-Pad8) -> Net-(U6-FB)
- U7 pad 1: /GPIO37 -> /GPIO47
- U7 pad 16: /ND2_2 -> +3V3
- U7 pad 26: /D1_2 -> GND
- U7 pad 8: unconnected-(U7-FB-Pad8) -> Net-(U7-FB)
Routing:
- net +3V3: track 307.6 -> 0.00 mm, vias 18 -> 0
- net /GPIO18: track 98.9 -> 0.00 mm, vias 2 -> 0
- net /GPIO38: track 87.0 -> 0.00 mm, vias 2 -> 0
- net /GPIO37: track 84.8 -> 0.00 mm, vias 2 -> 0
- net /GPIO1: track 65.2 -> 0.00 mm, vias 1 -> 0
- net /CASE: track 64.5 -> 0.00 mm, vias 2 -> 0
- net /D1_2: track 55.5 -> 0.00 mm, vias 2 -> 0
- net /SLEW_2: track 54.6 -> 0.00 mm, vias 2 -> 0
- net /ND2_2: track 54.4 -> 0.00 mm, vias 2 -> 0
- net /INV_2: track 51.9 -> 0.00 mm, vias 2 -> 0
- net /DISTANCE_R90_OUT: track 49.7 -> 0.00 mm, vias 1 -> 0
- net /DISTANCE_INTR: track 49.2 -> 0.00 mm, vias 1 -> 0
- net /ESP_BOOT: track 47.9 -> 0.00 mm, vias 2 -> 0
- net /SLEW_1: track 44.5 -> 0.00 mm, vias 4 -> 0
- net /DISTANCE_R_OUT: track 42.7 -> 0.00 mm, vias 1 -> 0
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- removed copper zone on B.Cu, net +3V3
- removed copper zone on F.Cu, net +3V3
- removed copper zone on In1.Cu, net +3V3
- removed copper zone on B.Cu, net +5V
- removed copper zone on F.Cu, net +5V
- removed copper zone on In1.Cu, net +5V
- removed copper zone on F.Cu, net +BATT
- removed copper zone on F.Cu, net /MOTOR1_A
- removed copper zone on In1.Cu, net /MOTOR1_A
- removed copper zone on F.Cu, net /MOTOR1_B
- removed copper zone on In1.Cu, net /MOTOR1_B
- removed copper zone on F.Cu, net /MOTOR2_A
- removed copper zone on In1.Cu, net /MOTOR2_A
- removed copper zone on F.Cu, net /MOTOR2_B
- removed copper zone on In1.Cu, net /MOTOR2_B
- removed copper zone on B.Cu, net GND
- removed copper zone on F.Cu, net GND
- removed copper zone on F.Cu, net Net-(D1-A)
- removed copper zone on F.Cu, net Net-(U1-SW)
Other:
- board size 40.1 x 90 mm -> 63 x 98 mm
- board text added: "- dimensiuni componente mai mari de 0603 - thermal relief-uri pe ground - condensatori de mai multe valori pe batt input ✅ - valori VOLTAGE condensatori x3 mai mari - piese corecte - spatiere mai mare intre componente - D1 - low, D2 - high, SLEW - floating, INV - floating, FB - rezistenta la GND ✅ - pad-urile de breakout sa fie la 3v3, fara rezistente - le am scos momentan - leduri mai putin pute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"
- board text removed: "-"
- board text removed: "- dimensiuni componente mai mari de 0603 - thermal relief-uri pe ground - condensatori de mai multe valori pe batt input - valori VOLTAGE condensatori x3 mai mari - piese corecte - spatiere mai mare intre componente - D1 - low, D2 - high, SLEW - floating, INV - floating, FB - rezistenta la GND - pad-urile de breakout sa fie la 3v3, fara rezistente - leduri mai putin puternice pt battery indicator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"
- board text removed: "1-INV_1 2-SLEW_1 3-D1_1 4-ND2_1 5-INV_2 6-SLEW_2 7-D1_2 8-ND2_2"
- board text removed: "2"
- board text removed: "3"
- board text removed: "3V3 ON"
- board text removed: "5"
- board text removed: "6"
- board text removed: "7"
- board text removed: "8"
- board text removed: "BATTERY LEVEL"
- board text removed: "BOOT"
- board text removed: "CASE"
- board text removed: "D1_1"
- board text removed: "D1_2"
- board text removed: "DIST_CENTER"
- board text removed: "DIST_L"
- board text removed: "DIST_L90"
- board text removed: "DIST_LF"
- board text removed: "DIST_R"
- board text removed: "DIST_R90"
- board text removed: "EN"
- board text removed: "INV_1"
- board text removed: "INV_2"
- board text removed: "IO13"
- board text removed: "IO21"
- board text removed: "IO47"
- board text removed: "IO48"
- board text removed: "LINE_L"
- board text removed: "LINE_R"
- board text removed: "MOTOR 1"
- board text removed: "MOTOR 2"
- board text removed: "ND2_1"
- board text removed: "ND2_2"
- board text removed: "PULLDOWN"
- board text removed: "PULLUP"
- board text removed: "SERVO"
- board text removed: "SLEW_1"
- board text removed: "SLEW_2"
- board text removed: "START MODULE"

Commit message: more testing
Parts:
- added C1: 0.1uF, Capacitor_SMD:C_0402_1005Metric, F.Cu at (95.1, 103.7)
- added C10: 47uF, Capacitor_SMD:C_1210_3225Metric, F.Cu at (142.8, 72.8)
- added C11: 100nF, Capacitor_SMD:C_0603_1608Metric, F.Cu at (152.1, 73.4)
- added C12: 0.1uF, Capacitor_SMD:C_0603_1608Metric, F.Cu at (79.4, 86.4)
- added C13: 1uF, Capacitor_SMD:C_0603_1608Metric, F.Cu at (162.4, 78.9)
- added C14: 10uF, Capacitor_SMD:C_0603_1608Metric, F.Cu at (153.2, 85.6)
- added C15: 10uF, Capacitor_SMD:C_0603_1608Metric, F.Cu at (147.6, 85.5)
- added C18: 0.1uF, Capacitor_SMD:C_0603_1608Metric, F.Cu at (79.4, 96.5)
- added C19: 33nF, Capacitor_SMD:C_0603_1608Metric, F.Cu at (79.4, 99.0)
- added C2: 10uF, Capacitor_SMD:C_0603_1608Metric, F.Cu at (79.4, 76.4)
- added C20: 33nF, Capacitor_SMD:C_0603_1608Metric, F.Cu at (79.4, 101.5)
- added C21: 100nF, Capacitor_SMD:C_0603_1608Metric, F.Cu at (83.4, 76.4)
- added C23: 100nF, Capacitor_SMD:C_0603_1608Metric, F.Cu at (83.4, 78.9)
- added C25: 0.1uF, Capacitor_SMD:C_0603_1608Metric, F.Cu at (83.4, 81.4)
- added C26: 0.1uF, Capacitor_SMD:C_0603_1608Metric, F.Cu at (83.4, 83.9)
- added C27: 100nF, Capacitor_SMD:C_0603_1608Metric, F.Cu at (83.4, 86.4)
- added C28: 100nF, Capacitor_SMD:C_0603_1608Metric, F.Cu at (83.4, 88.9)
- added C29: 0.1uF, Capacitor_SMD:C_0603_1608Metric, F.Cu at (83.4, 91.4)
- added C3: 0.1uF, Capacitor_SMD:C_0402_1005Metric, F.Cu at (161.5, 76.4)
- added C30: 0.1uF, Capacitor_SMD:C_0603_1608Metric, F.Cu at (76.9, 93.2)
- added C32: 1uF, Capacitor_SMD:C_0402_1005Metric, F.Cu at (95.1, 107.7)
- added C4: 10uF, Capacitor_SMD:C_1210_3225Metric, F.Cu at (149.4, 77.6)
- added C5: 220nF, Capacitor_SMD:C_0805_2012Metric, F.Cu at (152.1, 77.1)
- added C6: 0.1uF, Capacitor_SMD:C_0603_1608Metric, F.Cu at (79.4, 78.9)
- added C7: 0.1uF, Capacitor_SMD:C_0603_1608Metric, F.Cu at (79.4, 81.4)
- added C8: 47uF, Capacitor_SMD:C_1210_3225Metric, F.Cu at (149.4, 72.8)
- added C9: 47uF, Capacitor_SMD:C_1210_3225Metric, F.Cu at (146.1, 72.8)
- added D10: 2Vf, 20mA, RED, LED_SMD:LED_0603_1608Metric, F.Cu at (168.0, 100.3)
- added D11: LED_Small, LED_SMD:LED_0603_1608Metric, F.Cu at (123.1, 90.8)
- added D12: LED_Small, LED_SMD:LED_0603_1608Metric, F.Cu at (123.1, 77.1)
- added D13: LED_Small, LED_SMD:LED_0603_1608Metric, F.Cu at (123.1, 83.9)
- added D14: LED_Small, LED_SMD:LED_0603_1608Metric, F.Cu at (123.0, 113.5)
- added D15: LED_Small, LED_SMD:LED_0603_1608Metric, F.Cu at (123.0, 99.9)
- added D16: LED_Small, LED_SMD:LED_0603_1608Metric, F.Cu at (123.0, 106.7)
- added D17: LED_Small, LED_SMD:LED_0603_1608Metric, F.Cu at (109.1, 64.2)
- added D18: LED_Small, LED_SMD:LED_0603_1608Metric, F.Cu at (112.3, 122.8)
- added D2: 2Vf, 20mA, RED, LED_SMD:LED_0603_1608Metric, F.Cu at (99.5, 93.4)
- added D3: D_Schottky_Small, Diode_SMD:D_SOD-123, F.Cu at (100.4, 106.8)
- added D4: 10V, Diode_SMD:Nexperia_CFP3_SOD-123W, F.Cu at (90.9, 104.4)
- added D5: 8.2V, Diode_SMD:Nexperia_CFP3_SOD-123W, F.Cu at (90.9, 107.6)
- added D6: 6V, Diode_SMD:Nexperia_CFP3_SOD-123W, F.Cu at (90.9, 110.9)
- added D7: 2Vf, 20mA, RED, LED_SMD:LED_0603_1608Metric, F.Cu at (99.5, 96.0)
- added D8: 2Vf, 20mA, RED, LED_SMD:LED_0603_1608Metric, F.Cu at (99.5, 98.6)
- added D9: 2Vf, 20mA, RED, LED_SMD:LED_0603_1608Metric, F.Cu at (107.4, 108.8)
- added JP1: SolderJumper_3_Open, Jumper:SolderJumper-3_P1.3mm_Open_RoundedPad1.0x1.5mm_NumberLabels, F.Cu at (105.9, 76.9)
- added JP2: SolderJumper_3_Open, Jumper:SolderJumper-3_P1.3mm_Open_RoundedPad1.0x1.5mm_NumberLabels, F.Cu at (105.9, 80.5)
- added JP3: SolderJumper_3_Open, Jumper:SolderJumper-3_P1.3mm_Open_RoundedPad1.0x1.5mm_NumberLabels, F.Cu at (105.9, 84.0)
- added JP4: SolderJumper_3_Open, Jumper:SolderJumper-3_P1.3mm_Open_RoundedPad1.0x1.5mm_NumberLabels, F.Cu at (105.9, 87.5)
- added R1: 10k, Resistor_SMD:R_0603_1608Metric, F.Cu at (83.4, 96.5)
- added R10: 1k, Resistor_SMD:R_0603_1608Metric, F.Cu at (87.4, 91.4)
- added R11: 1k, Resistor_SMD:R_0603_1608Metric, F.Cu at (87.4, 94.0)
- added R12: 1k, Resistor_SMD:R_0603_1608Metric, F.Cu at (87.4, 96.5)
- added R13: 10k, Resistor_SMD:R_0603_1608Metric, F.Cu at (87.4, 99.0)
- added R14: 10k, Resistor_SMD:R_0603_1608Metric, F.Cu at (87.4, 101.5)
- added R15: 10k, Resistor_SMD:R_0603_1608Metric, F.Cu at (91.5, 76.4)
- added R16: 10k, Resistor_SMD:R_0603_1608Metric, F.Cu at (91.5, 78.9)
- added R17: 412, Resistor_SMD:R_0603_1608Metric, F.Cu at (91.5, 81.4)
- added R18: 300, Resistor_SMD:R_0603_1608Metric, F.Cu at (91.5, 83.9)
- added R19: 68, Resistor_SMD:R_0603_1608Metric, F.Cu at (164.8, 100.3)
- added R2: 5k1, Resistor_SMD:R_0603_1608Metric, F.Cu at (83.4, 99.0)
- added R20: ?, Resistor_SMD:R_0603_1608Metric, F.Cu at (123.1, 87.8)
- added R21: 2k, Resistor_SMD:R_0603_1608Metric, F.Cu at (112.1, 61.1)
- added R22: 3.3k, Resistor_SMD:R_0603_1608Metric, F.Cu at (109.1, 61.1)
- added R23: 2k, Resistor_SMD:R_0603_1608Metric, F.Cu at (109.2, 124.4)
- added R24: 3.3k, Resistor_SMD:R_0603_1608Metric, F.Cu at (112.3, 124.5)
- added R25: 200, Resistor_SMD:R_0603_1608Metric, F.Cu at (110.0, 108.4)
- added R26: ?, Resistor_SMD:R_0603_1608Metric, F.Cu at (123.1, 74.1)
- added R27: ?, Resistor_SMD:R_0603_1608Metric, F.Cu at (123.1, 80.9)
- added R28: ?, Resistor_SMD:R_0603_1608Metric, F.Cu at (123.0, 110.5)
- added R29: ?, Resistor_SMD:R_0603_1608Metric, F.Cu at (123.0, 96.9)
- added R3: 5k1, Resistor_SMD:R_0603_1608Metric, F.Cu at (83.4, 101.5)
- added R30: ?, Resistor_SMD:R_0603_1608Metric, F.Cu at (123.0, 103.7)
- added R31: ?, Resistor_SMD:R_0603_1608Metric, F.Cu at (112.1, 64.2)
- added R32: ?, Resistor_SMD:R_0603_1608Metric, F.Cu at (109.2, 122.8)
- added R4: 100k, Resistor_SMD:R_0603_1608Metric, F.Cu at (158.9, 83.3)
- added R5: 22.1k, Resistor_SMD:R_0603_1608Metric, F.Cu at (158.9, 81.7)
- added R6: 68, Resistor_SMD:R_0603_1608Metric, F.Cu at (87.4, 81.4)
- added R7: 10k, Resistor_SMD:R_0603_1608Metric, F.Cu at (87.4, 83.9)
- added R8: 5k, Resistor_SMD:R_0603_1608Metric, F.Cu at (87.4, 86.4)
- added R9: 1k, Resistor_SMD:R_0603_1608Metric, F.Cu at (87.4, 88.9)
- added TP1: GPIO13, TestPoint:TestPoint_Pad_1.5x1.5mm, F.Cu at (79.2, 104.5)
- added TP10: SLEW_2, TestPoint:TestPoint_Pad_1.5x1.5mm, F.Cu at (82.7, 111.6)
- added TP11: INV_2, TestPoint:TestPoint_Pad_1.5x1.5mm, F.Cu at (86.3, 104.5)
- added TP12: GPIO37, TestPoint:TestPoint_Pad_1.5x1.5mm, F.Cu at (86.3, 108.1)
- added TP13: GPIO48, TestPoint:TestPoint_Pad_1.5x1.5mm, F.Cu at (86.3, 111.6)
- added TP6: SLEW_1, TestPoint:TestPoint_Pad_1.5x1.5mm, F.Cu at (79.2, 108.1)
- added TP7: INV_1, TestPoint:TestPoint_Pad_1.5x1.5mm, F.Cu at (79.2, 111.6)
- added TP8: GPIO35, TestPoint:TestPoint_Pad_1.5x1.5mm, F.Cu at (82.7, 104.5)
- added TP9: GPIO36, TestPoint:TestPoint_Pad_1.5x1.5mm, F.Cu at (82.7, 108.1)
- C31: footprint Capacitor_SMD:C_1210_3225Metric -> Capacitor_SMD:C_0603_1608Metric
- moved L1 72.4 mm to (157.1, 71.7), turned to 180 degrees
- moved U1 57.8 mm to (157.1, 78.2)
- moved SW1 55.5 mm to (100.9, 50.7)
- moved SW5 45.2 mm to (97.0, 56.5)
- moved D1 40.8 mm to (155.9, 102.1)
- moved U4 30.6 mm to (150.4, 85.5)
- moved C33 29.6 mm to (144.4, 108.9)
- moved SW2 26.4 mm to (167.1, 86.8)
- moved U6 22.2 mm to (131.4, 86.8), turned to 180 degrees
- moved U7 21.5 mm to (131.7, 100.2), turned to 180 degrees
- moved J6 20.9 mm to (137.7, 115.6), turned to 0 degrees
- moved U2 20.2 mm to (159.7, 94.0)
- moved J1 20.0 mm to (166.4, 94.0)
- moved C31 15.2 mm to (140.5, 111.6)
- moved J8 12.5 mm to (127.9, 128.1), turned to 180 degrees
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Connections:
- U2 pad 1: /D+ -> /D-
- U2 pad 3: /D- -> /D+
- U2 pad 4: /D_N -> /D_P
- U2 pad 6: /D_P -> /D_N
Routing:
- net /D_P: track 0.00 -> 2.24 mm
- net /D_N: track 0.00 -> 2.24 mm
Other:
- board size 63 x 98 mm -> 62.4 x 98 mm

Commit message: another variant
Parts:
- removed C25, C26: 0.1uF, Capacitor_SMD:C_0603_1608Metric
- C1, C3: footprint Capacitor_SMD:C_0402_1005Metric -> Capacitor_SMD:C_0603_1608Metric
- moved C6 83.4 mm to (160.6, 98.1), turned to -90 degrees
- moved C18 83.2 mm to (161.9, 85.8)
- moved R3 78.0 mm to (160.6, 90.4), turned to -90 degrees
- moved R10 76.6 mm to (163.2, 103.1)
- moved TP8 75.8 mm to (158.4, 109.0)
- moved TP10 75.7 mm to (158.3, 116.2)
- moved TP7 75.7 mm to (154.8, 116.2)
- moved TP1 75.7 mm to (154.8, 109.0)
- moved TP13 75.7 mm to (161.8, 116.2)
- moved TP6 75.7 mm to (154.8, 112.6)
- moved TP9 75.7 mm to (158.3, 112.6)
- moved TP11 75.7 mm to (161.8, 109.0)
- moved TP12 75.7 mm to (161.8, 112.6)
- moved R2 74.7 mm to (158.1, 97.3)
- moved R8 74.7 mm to (162.1, 87.6)
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Connections:
- JP1 pad 3: +5V -> +3V3
- JP2 pad 3: +5V -> +3V3
- JP3 pad 3: +5V -> +3V3
- JP4 pad 3: +5V -> +3V3
Routing:
- net /D-: track 0.00 -> 66.6 mm, vias 0 -> 2
- net /D+: track 0.00 -> 66.3 mm, vias 0 -> 2

Commit message: final test layout
Routing:
- net /D-: track 66.6 -> 56.9 mm
- net /D+: track 66.3 -> 56.9 mm

Commit message: another variant
Parts:
- added C44: 100nF, Capacitor_SMD:C_0603_1608Metric, F.Cu at (122.2, 75.7)
- added C45: 100nF, Capacitor_SMD:C_0603_1608Metric, F.Cu at (122.2, 81.3)
- added C46: 100nF, Capacitor_SMD:C_0603_1608Metric, F.Cu at (122.2, 88.0)
- added C47: 100nF, Capacitor_SMD:C_0603_1608Metric, F.Cu at (122.1, 97.1)
- added C48: 100nF, Capacitor_SMD:C_0603_1608Metric, F.Cu at (122.1, 103.9)
- added C49: 100nF, Capacitor_SMD:C_0603_1608Metric, F.Cu at (122.1, 111.0)
- C32: footprint Capacitor_SMD:C_0402_1005Metric -> Capacitor_SMD:C_0603_1608Metric
- moved SW1 76.0 mm to (150.4, 114.7)
- moved C7 73.1 mm to (152.9, 114.6), turned to 90 degrees
- moved C32 71.3 mm to (147.9, 116.2), turned to 90 degrees
- moved C12 71.1 mm to (158.0, 116.2)
- moved SW5 71.0 mm to (155.5, 114.8)
- moved R1 68.4 mm to (147.9, 113.2)
- moved R7 67.7 mm to (158.0, 113.3), turned to -90 degrees
- moved C2 61.8 mm to (164.5, 81.6)
- moved C1 61.5 mm to (164.5, 83.1)
- moved C14 54.9 mm to (114.7, 46.5)
- moved C15 54.9 mm to (109.1, 46.4)
- moved U4 54.9 mm to (111.9, 46.4)
- moved U3 50.4 mm to (156.5, 93.7), turned to -90 degrees
- moved TP10 45.6 mm to (140.6, 74.1)
- moved R4 44.8 mm to (119.1, 62.7), turned to 90 degrees
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Connections:
- U2 pad 1: /D- -> /D+
- U2 pad 3: /D+ -> /D-
- U2 pad 4: /D_P -> /D_N
- U2 pad 6: /D_N -> /D_P
Routing:
- net /D-: track 56.9 -> 11.4 mm, vias 2 -> 0
- net /D+: track 56.9 -> 12.2 mm, vias 2 -> 0
- net /D_P: track 2.24 -> 6.60 mm
- net /D_N: track 2.24 -> 5.52 mm
- added copper zone on B.Cu, net GND
- added copper zone on In1.Cu, net GND

Commit message: backup with layout
Parts:
- added C10: 47uF, Capacitor_SMD:C_1210_3225Metric, F.Cu at (161.6, 39.9)
- added C11: 100nF, Capacitor_SMD:C_0603_1608Metric, F.Cu at (162.3, 49.5)
- added C13: 1uF, Capacitor_SMD:C_0603_1608Metric, F.Cu at (157.7, 59.7)
- added C25: 100nF, Capacitor_SMD:C_0603_1608Metric, F.Cu at (136.4, 86.4)
- added C26: 100nF, Capacitor_SMD:C_0603_1608Metric, F.Cu at (133.4, 95.4)
- added C3: 0.1uF, Capacitor_SMD:C_0402_1005Metric, F.Cu at (159.8, 58.8)
- added C34: 100nF, Capacitor_SMD:C_0603_1608Metric, F.Cu at (131.9, 106.5)
- added C35: 100nF, Capacitor_SMD:C_0603_1608Metric, F.Cu at (132.7, 92.4)
- added C4: 10uF, Capacitor_SMD:C_1210_3225Metric, F.Cu at (156.9, 46.6)
- added C5: 220nF, Capacitor_SMD:C_0805_2012Metric, F.Cu at (159.1, 49.5)
- added C8: 47uF, Capacitor_SMD:C_1210_3225Metric, F.Cu at (161.6, 43.2)
- added C9: 47uF, Capacitor_SMD:C_1210_3225Metric, F.Cu at (161.6, 46.7)
- added L1: 10uH, 27mOhm, footprints:IND_XAL6060-103MEC, F.Cu at (165.3, 55.0)
- added R4: 100k, Resistor_SMD:R_0402_1005Metric, F.Cu at (154.0, 56.5)
- added R5: 22.1k, Resistor_SMD:R_0402_1005Metric, F.Cu at (155.1, 56.5)
- added U1: LMR33630ADDAR, footprints:DDA0008J, F.Cu at (158.4, 54.3)
- moved C21 12.5 mm to (132.0, 80.5), turned to 90 degrees
- moved C31 12.1 mm to (128.4, 109.7), turned to 180 degrees
- moved R14 11.3 mm to (136.3, 82.5), turned to -90 degrees
- moved TP12 10.0 mm to (160.7, 107.0)
- moved C29 9.85 mm to (133.0, 78.2), turned to 0 degrees
- moved TP13 7.60 mm to (153.2, 107.0)
- moved R16 6.26 mm to (135.6, 96.8), turned to -90 degrees
- moved J6 5.50 mm to (143.2, 115.6), turned to 180 degrees
- moved C30 5.17 mm to (128.0, 78.3)
- moved C27 4.17 mm to (138.2, 93.1)
- moved R29 3.48 mm to (122.2, 100.2), turned to 90 degrees
- moved R19 3.40 mm to (168.2, 95.3), turned to 90 degrees
- moved R27 3.32 mm to (123.7, 84.3), turned to 90 degrees
- moved R26 3.24 mm to (123.7, 77.4), turned to 90 degrees
- moved R30 3.03 mm to (123.5, 106.8), turned to 90 degrees
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Routing:
- net /GPIO1: track 0.00 -> 70.6 mm, vias 0 -> 1
- net /DISTANCE_L90_OUT: track 0.00 -> 56.7 mm
- net /GPIO18: track 0.00 -> 56.4 mm, vias 0 -> 1
- net /INV_2: track 0.00 -> 50.9 mm, vias 0 -> 4
- net /GPIO8: track 0.00 -> 49.6 mm, vias 0 -> 1
- net /DISTANCE_LF_OUT: track 0.00 -> 49.1 mm
- net /DISTANCE_INTR: track 0.00 -> 44.8 mm
- net /GPIO10: track 0.00 -> 43.0 mm
- net /GPIO11: track 0.00 -> 41.2 mm
- net /DISTANCE_L_OUT: track 0.00 -> 40.3 mm
- net /GPIO12: track 0.00 -> 39.2 mm
- net /SLEW_2: track 0.00 -> 38.0 mm, vias 0 -> 4
- net /DISTANCE_R90: track 0.00 -> 33.0 mm, vias 0 -> 2
- net /DISTANCE_R_OUT: track 0.00 -> 32.3 mm
- net /DISTANCE_R: track 0.00 -> 30.9 mm, vias 0 -> 2
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- added copper zone on F.Cu, net +BATT
- added copper zone on In2.Cu, net +BATT
- added copper zone on B.Cu, net /MOTOR1_A
- added copper zone on F.Cu, net /MOTOR1_A
- added copper zone on B.Cu, net /MOTOR1_B
- added copper zone on F.Cu, net /MOTOR1_B
- added copper zone on B.Cu, net /MOTOR2_A
- added copper zone on F.Cu, net /MOTOR2_A
- added copper zone on F.Cu, net Net-(D1-A)
- added copper zone on F.Cu, net Net-(U1-SW)
