File: minisumo_2025.kicad_sch (KiCad schematic)
At the start: 119 parts, among them J1 USB_C Connector, J10 DISTANCE_R90, J11 DISTANCE_R, J12 DISTANCE_RF, J13 DISTANCE_L90, J14 DISTANCE_L, J15 LINE_LEFT, J16 DISTANCE_LF, J3 START_MODULE, J4 MOTOR1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

Commit message: more testing
Parts:
- C31: footprint Capacitor_SMD:C_1210_3225Metric -> Capacitor_SMD:C_0603_1608Metric
Connections:
- net D+: now also U2.3 (I/O2); no longer U2.1 (I/O1)
- net D-: now also U2.1 (I/O1); no longer U2.3 (I/O2)
- net D_N: now also U2.6 (I/O1); no longer U2.4 (I/O2)
- net D_P: now also U2.4 (I/O2); no longer U2.6 (I/O1)
Changed lines of the file:
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@@
 		)
 	)
+	(label "D_P"
+		(at 118.11 52.07 0)
+		(effects
+			(font
+				(size 1.27 1.27)
+			)
+			(justify left bottom)
+		)
+	)
 	(label "LINE_LEFT"
 		(at 139.7 271.78 180)
@@
 		)
 	)
-	(label "D_P"
-		(at 118.11 49.53 0)
-		(effects
-			(font
-				(size 1.27 1.27)
-			)
-			(justify left bottom)
-		)
-	)
 	(label "MOTOR1_A"
 		(at 83.82 147.32 180)
@@
 		)
 	)
+	(label "D-"
+		(at 104.14 49.53 0)
+		(effects
+			(font
+				(size 1.27 1.27)
+			)
+			(justify left bottom)
+		)
+	)
 	(label "LINE_RIGHT"
 		(at 360.68 62.23 0)
@@
 		)
 	)
+	(label "D_N"
+		(at 118.11 49.53 0)
+		(effects
+			(font
+				(size 1.27 1.27)
+			)
+			(justify left bottom)
+		)
+	)
 	(label "GPIO37"
 		(at 86.36 57.15 0)
@@
 		)
 	)
-	(label "D+"
-		(at 104.14 49.53 0)
-		(effects
-			(font
-				(size 1.27 1.27)
-			)
-			(justify left bottom)
-		)
-	)
 	(label "INDICATOR_LED"
 		(at 360.68 52.07 0)
@@
 		)
 	)
+	(label "D+"
+		(at 104.14 52.07 0)
+		(effects
+			(font
+				(size 1.27 1.27)
+			)
+			(justify left bottom)
+		)
+	)
 	(label "LINE_LEFT_OUT"
 		(at 119.38 271.78 180)
@@
 		)
 	)
-	(label "D_N"
-		(at 118.11 52.07 0)
-		(effects
-			(font
-				(size 1.27 1.27)
-			)
-			(justify left bottom)
-		)
-	)
 	(label "GPIO47"
 		(at 355.6 77.47 180)
@@
 		)
 	)
-	(label "D-"
-		(at 104.14 52.07 0)
-		(effects
-			(font
-				(size 1.27 1.27)
-			)
-			(justify left bottom)
-		)
-	)
 	(label "DISTANCE_LF_OUT"
 		(at 233.68 232.41 180)
@@
 			)
 		)
-		(property "Footprint" "Capacitor_SMD:C_1210_3225Metric"
+		(property "Footprint" "Capacitor_SMD:C_0603_1608Metric"
 			(at 175.26 77.47 0)
 			(effects

Commit message: another variant
Parts:
- removed C25, C26: 0.1uF, Capacitor_SMD:C_0603_1608Metric, symbol Device:C_Small
- C1, C3: footprint Capacitor_SMD:C_0402_1005Metric -> Capacitor_SMD:C_0603_1608Metric
Connections:
- net +3V3: now also JP1.3 (B), JP2.3 (B), JP3.3 (B), JP4.3 (B)
- net +5V: no longer JP1.3 (B), JP2.3 (B), JP3.3 (B), JP4.3 (B)

Commit message: another variant
Parts:
- added C44, C45, C46, C47, C48, C49: 100nF, Capacitor_SMD:C_0603_1608Metric, symbol Device:C_Small
- C32: footprint Capacitor_SMD:C_0402_1005Metric -> Capacitor_SMD:C_0603_1608Metric
Connections:
- net +5V: now also C44.1, C45.1, C46.1, C47.1, C48.1, C49.1
- net D+: now also U2.1 (I/O1); no longer U2.3 (I/O2)
- net D-: now also U2.3 (I/O2); no longer U2.1 (I/O1)
- net D_N: now also U2.4 (I/O2); no longer U2.6 (I/O1)
- net D_P: now also U2.6 (I/O1); no longer U2.4 (I/O2)
- net GND: now also C44.2, C45.2, C46.2, C47.2, C48.2, C49.2

Commit message: routing
Parts:
- added C25: 100nF, Capacitor_SMD:C_0603_1608Metric, symbol Device:C_Small
- TP13: value GPIO48 -> GPIO17
Connections:
- net +BATT: now also C25.1
- net DISTANCE_INTR: now also U3.22 (IO14); no longer U3.17 (IO9)
- net DISTANCE_L: now also U3.8 (IO15); no longer U3.5 (IO5)
- net DISTANCE_L90: now also U3.9 (IO16); no longer U3.4 (IO4)
- net DISTANCE_LF: now also U3.7 (IO7); no longer U3.6 (IO6)
- net DISTANCE_R: now also U3.5 (IO5); no longer U3.8 (IO15)
- net DISTANCE_R90: now also U3.4 (IO4); no longer U3.9 (IO16)
- net DISTANCE_RF: now also U3.6 (IO6); no longer U3.7 (IO7)
- net GND: now also C25.2
- net GPIO10: now also U6.1 (IN2); no longer J8.5 (Pin_5)
- net GPIO11: now also U7.2 (IN1); no longer J8.4 (Pin_4)
- net GPIO12: now also U7.1 (IN2); no longer J8.3 (Pin_3)
- net GPIO17: now also TP13.1; no longer U6.1 (IN2)
- net GPIO21: now also J8.5 (Pin_5); no longer U6.2 (IN1)
- net GPIO38: now also R19.1; no longer U7.2 (IN1)
- net GPIO47: now also J8.4 (Pin_4); no longer U7.1 (IN2)
- net GPIO48: now also J8.3 (Pin_3); no longer TP13.1
- removed net GPIO14: R19.1, U3.22 (IO14)
- new net GPIO9: U3.17 (IO9), U6.2 (IN1)
Other:
- moved on the sheet: TP13

Commit message: layout done
Parts:
- added C16: 0.1uF, Capacitor_SMD:C_0603_1608Metric, symbol Device:C_Small
Connections:
- net DISTANCE_L: now also U3.6 (IO6), U5.6 (A5); no longer U3.8 (IO15), U5.3 (A2)
- net DISTANCE_L90: now also U3.4 (IO4), U5.8 (A7); no longer U3.9 (IO16), U5.1 (A1)
- net DISTANCE_L90_OUT: now also U5.13 (B7); no longer U5.20 (B1)
- net DISTANCE_LF: now also U3.5 (IO5), U5.7 (A6); no longer U3.7 (IO7), U5.4 (A3)
- net DISTANCE_LF_OUT: now also U5.14 (B6); no longer U5.17 (B3)
- net DISTANCE_L_OUT: now also U5.15 (B5); no longer U5.18 (B2)
- net DISTANCE_R: now also U3.7 (IO7), U5.4 (A3); no longer U3.5 (IO5), U5.7 (A6)
- net DISTANCE_R90: now also U3.8 (IO15), U5.3 (A2); no longer U3.4 (IO4), U5.8 (A7)
- net DISTANCE_R90_OUT: now also U5.18 (B2); no longer U5.13 (B7)
- net DISTANCE_RF: now also U3.9 (IO16), U5.1 (A1); no longer U3.6 (IO6), U5.6 (A5)
- net DISTANCE_RF_OUT: now also U5.20 (B1); no longer U5.15 (B5)
- net DISTANCE_R_OUT: now also U5.17 (B3); no longer U5.14 (B6)
- net GND: now also C16.2
- net at C6.1, D3.2 (A), J1.A4 (VBUS)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: now also C16.1

Commit message: more changes
Parts:
- C11: value 100nF -> 0.1uF
- D5: value 8.2V -> 8V
- R17: value 412 -> 7k5
- R18: value 300 -> 5k5
- R19: value 68 -> 1k
- R20, R26, R27, R28, R29, R30, R31, R32: value ? -> 3k3
- R25: value 200 -> 3k3
Other:
- note added: "All LEDs are GREEN, 5mA, 2.5fV, 0603"
- note removed: "TODO:"
- moved on the sheet: D10, R19, TP1, TP12, TP13, TP8, TP9

Commit message: final layout
Parts:
- removed D1: D_Schottky_Small, Diode_SMD:D_SOD-123, symbol Device:D_Schottky_Small
- added C17, C26: 0.1uF, Capacitor_SMD:C_0603_1608Metric, symbol Device:C_Small
- added FB1: FerriteBead_Small, Capacitor_SMD:C_0805_2012Metric, symbol Device:FerriteBead_Small
- added Q1: Si2371EDS, Package_TO_SOT_SMD:SOT-23, symbol Transistor_FET:Si2371EDS
- D3: LCSC Part # C389355 -> (none)
Connections:
- net +5V: now also Q1.2 (S); no longer U2.5 (VBUS)
- net GND: now also C17.2, C26.2
- net at C10.2, C11.2, C8.2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: now also Q1.3 (D)
- net at C16.1, J1.A4 (VBUS), J1.A9 (VBUS)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: now also C17.1, FB1.1; no longer C6.1, D3.2 (A)
- new net VBUS: C26.1, C6.1, D3.2 (A), FB1.2, Q1.1 (G), U2.5 (VBUS)
Other:
- moved on the sheet: C10, C11, C13, C14, C15, C16, C3, C31, C33, C4, C5, C6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

Commit message: silksreen and bom
Parts:
- removed SW5: BOOT, footprints:SW_TS-1088-AR02016, symbol Switch:SW_Push_Dual_x2
- added C34: 0.1uF, Capacitor_SMD:C_0603_1608Metric, symbol Device:C_Small
- added SW3: BOOT, footprints:435441019830, symbol Switch:SW_Push_Dual_x2
- C1, C11, C12, C16, C17, C18, C26, C29, C30, C6, C7: M_NUMBER (none) -> 810-CGA3E2X7R1H104K
- C10, C8, C9: M_NUMBER (none) -> 81-GRM32ER61C476KE5L
- C13, C32: M_NUMBER (none) -> 80-C0603C105K8P
- C14, C15, C2: M_NUMBER (none) -> 810-CGA3EDX7T1A106M0
- C19, C20: M_NUMBER (none) -> 81-GCM188R71H333JA5D
- C21, C23, C25, C27, C28, C44, C45, C46, C47, C48, C49: value 100nF -> 0.1uF; M_NUMBER (none) -> 810-CGA3E2X7R1H104K
- C22, C24: value 100uF -> 100uF - low ESR; M_NUMBER (none) -> -
- C3: M_NUMBER (none) -> 80-C0603C104M4RAC
- C31: M_NUMBER (none) -> 81-GRM188R6YA475KE5D
- C33, J10, J11, J12, J13, J14, J15, J16, J3, J4, J5, J6, J8, J9, TP1, TP10, TP11, TP12, TP13, TP6, TP7, TP8, TP9: M_NUMBER (none) -> -
- C4: M_NUMBER (none) -> 810-C3225X7R1H106MAC
- C5: M_NUMBER (none) -> 810-C2012X7R1H224K
- D10: value 2Vf, 20mA, RED -> LED_Small; M_NUMBER (none) -> 720-P4112S2U1252X4X5
- D11, D12, D13, D14, D15, D16, D17, D18: M_NUMBER (none) -> 720-P4112S2U1252X4X5
- D2, D7, D8, D9: value 2Vf, 20mA, RED -> 1.95Vf, 20mA, RED; M_NUMBER (none) -> 720-P412Q1S136A8J802
- D3: M_NUMBER (none) -> 241-SS0530_R1_00001
- D4: footprint Diode_SMD:Nexperia_CFP3_SOD-123W -> Diode_SMD:D_SOD-123F; M_NUMBER (none) -> 771-BZT52H-A10-QX
- D5: value 8V -> 8.2V; footprint Diode_SMD:Nexperia_CFP3_SOD-123W -> Diode_SMD:D_SOD-123F; M_NUMBER (none) -> 771-BZT52H-C8V2115
- D6: value 6V -> 6.2V; footprint Diode_SMD:Nexperia_CFP3_SOD-123W -> Diode_SMD:D_SOD-123F; M_NUMBER (none) -> 771-BZT52H-C6V2-QX
- FB1: M_NUMBER (none) -> BLM21PG121SN1D
- J1: M_NUMBER (none) -> 640-USB4215-03-A
- L1: value 10uH, 27mOhm -> 8.2uH, 21mOhm; footprint footprints:IND_XAL6060-103MEC -> Inductor_SMD:L_Coilcraft_XAL4040-XXX; M_NUMBER (none) -> 994-XAL4040-822MEC
- Q1: M_NUMBER (none) -> 78-SI2371EDS-T1-GE3
- R1, R13, R14, R15, R16, R7: M_NUMBER (none) -> 603-RC0603FR-0710KL
- R10, R11, R12, R19, R9: M_NUMBER (none) -> 603-RC0603FR-071KL
- R17: value 7k5 -> 5k; M_NUMBER (none) -> 603-RC0603FR-077K5L
- R18: value 5k5 -> 3k74; M_NUMBER (none) -> 71-CRCW06033K74DHEAP
- R2, R3: M_NUMBER (none) -> 603-RC0603FR-135K1L
- R20, R26, R27, R28, R29, R30, R31, R32: M_NUMBER (none) -> 603-RC0603FR-073K3L
- R21, R23: M_NUMBER (none) -> 603-RC0603FR-072KL
- R22, R24: value 3.3k -> 3k3; M_NUMBER (none) -> 603-RC0603FR-073K3L
- R25: value 3k3 -> 2k; M_NUMBER (none) -> 603-RC0603FR-073K3L
- R4: M_NUMBER (none) -> 603-RC0603FR-07100KL
- R5: value 22.1k -> 24k9; M_NUMBER (none) -> 603-RC0603FR-1324K9L
- R6: value 68 -> 1k; M_NUMBER (none) -> 603-RC0603FR-071KL
- R8: M_NUMBER (none) -> 303-0603SAF430KT5E
- SW1, SW2: footprint footprints:SW_TS-1088-AR02016 -> footprints:435441019830; M_NUMBER (none) -> 710-435441019830
- U1: M_NUMBER (none) -> 595-LMR33630ADDAR
- U2: M_NUMBER (none) -> 511-USBLC6-2P6
- U3: M_NUMBER (none) -> 356-ESP32S3WROOM1UN4
- U4: M_NUMBER (none) -> 595-TLV75733PDBVR
- U5: M_NUMBER (none) -> 595-TXS0108EPWR
- U6, U7: M_NUMBER (none) -> C3225X7R1H106M250AC
Connections:
- net +BATT: now also C34.1
- net CASE: now also SW2.3 (C)
- net ESP_BOOT: now also SW3.2 (D), SW3.3 (C)
- net ESP_EN: now also SW1.3 (C)
- net GND: now also SW1.4 (C), SW2.4 (C), C34.2, SW3.1 (C), SW3.4 (C)
