File: leds.kicad_sch (KiCad schematic)
At the start: 29 parts

Commit message: added global labels
Parts:
- removed D10, D11, D12, D13, D14, D15, D16, D17, D18: LED_Small, LED_SMD:LED_0603_1608Metric, symbol Device:LED_Small
- removed D2, D7, D8, D9: 1.95Vf, 20mA, RED, LED_SMD:LED_0603_1608Metric, symbol Device:LED_Small
- removed D4: 10V, Diode_SMD:D_SOD-123F, symbol Device:D_Zener_Small
- removed D5: 8.2V, Diode_SMD:D_SOD-123F, symbol Device:D_Zener_Small
- removed D6: 6.2V, Diode_SMD:D_SOD-123F, symbol Device:D_Zener_Small
- removed R17: 5k, Resistor_SMD:R_0603_1608Metric, symbol Device:R_Small
- removed R18: 3k74, Resistor_SMD:R_0603_1608Metric, symbol Device:R_Small
- removed R19, R6: 1k, Resistor_SMD:R_0603_1608Metric, symbol Device:R_Small
- removed R20, R26, R27, R28, R29, R30, R31, R32: 3k3, Resistor_SMD:R_0603_1608Metric, symbol Device:R_Small
- removed R25: 2k, Resistor_SMD:R_0603_1608Metric, symbol Device:R_Small
Other:
- note removed: "All LEDs are GREEN, 5mA, 2.5fV, 0603"
- note removed: "Power ON Led"
- note removed: "Sensor indicator leds"
