File: kicad/drivers.kicad_sch (KiCad schematic)
At the start: 32 parts, among them J4 MOTOR1, J5 MOTOR2, U6 MC33926PNB, U7 MC33926PNB

Commit message: 2026 version
Parts:
- removed JP1, JP2, JP3, JP4: SolderJumper_3_Open, Jumper:SolderJumper-3_P1.3mm_Open_RoundedPad1.0x1.5mm_NumberLabels, symbol Jumper:SolderJumper_3_Open
- removed R10, R11, R12, R9: 1k, Resistor_SMD:R_0603_1608Metric, symbol Device:R_Small
- removed TP10: SLEW_2, TestPoint:TestPoint_Pad_1.5x1.5mm, symbol Connector:TestPoint
- removed TP11: INV_2, TestPoint:TestPoint_Pad_1.5x1.5mm, symbol Connector:TestPoint
- removed TP6: SLEW_1, TestPoint:TestPoint_Pad_1.5x1.5mm, symbol Connector:TestPoint
- removed TP7: INV_1, TestPoint:TestPoint_Pad_1.5x1.5mm, symbol Connector:TestPoint
