File: kicad/sensors.kicad_sch (KiCad schematic)
At the start: 38 parts, among them J10 DISTANCE_R90, J11 DISTANCE_R, J12 DISTANCE_RF, J13 DISTANCE_L90, J14 DISTANCE_L, J15 LINE_LEFT, J16 DISTANCE_LF, J8 DISTANCE_CENTER, J9 LINE_RIGHT, U5 TXS0108EPWR

Commit message: 2026 version
Parts:
- removed C44, C45, C46, C47, C48, C49: 0.1uF, Capacitor_SMD:C_0603_1608Metric, symbol Device:C_Small
- removed D16: LED_Small, LED_SMD:LED_0603_1608Metric, symbol Device:LED_Small
- removed J10: DISTANCE_R90, footprints:CONN-TH_S3B-ZR-3.4-LF-SN, symbol Connector:Conn_01x03_Socket
- removed J11: DISTANCE_R, footprints:CONN-TH_S3B-ZR-3.4-LF-SN, symbol Connector:Conn_01x03_Socket
- removed J12: DISTANCE_RF, footprints:CONN-TH_S3B-ZR-3.4-LF-SN, symbol Connector:Conn_01x03_Socket
- removed J13: DISTANCE_L90, footprints:CONN-TH_S3B-ZR-3.4-LF-SN, symbol Connector:Conn_01x03_Socket
- removed J14: DISTANCE_L, footprints:CONN-TH_S3B-ZR-3.4-LF-SN, symbol Connector:Conn_01x03_Socket
- removed J15: LINE_LEFT, footprints:CONN-TH_S3B-ZR-3.4-LF-SN, symbol Connector:Conn_01x03_Socket
- removed J16: DISTANCE_LF, footprints:CONN-TH_S3B-ZR-3.4-LF-SN, symbol Connector:Conn_01x03_Socket
- removed J8: DISTANCE_CENTER, footprints:CONN-TH_S6B-ZR-3.4-LF-SN, symbol Connector:Conn_01x06_Socket
- removed J9: LINE_RIGHT, footprints:CONN-TH_S3B-ZR-3.4-LF-SN, symbol Connector:Conn_01x03_Socket
- removed R30: 3k3, Resistor_SMD:R_0603_1608Metric, symbol Device:R_Small
- added J2, J7: Conn_01x06_Pin, Connector_PinHeader_2.54mm:PinHeader_2x03_P2.54mm_Vertical, symbol Connector:Conn_01x06_Pin
- added J8: Conn_01x03_Pin, Connector_PinHeader_2.54mm:PinHeader_1x03_P2.54mm_Vertical, symbol Connector:Conn_01x03_Pin
Connections:
- net +3V3: now also J8.2 (Pin_2)
- net +5V: now also J2.2 (Pin_2), J7.2 (Pin_2)
- net DISTANCE_L90_OUT: now also J7.3 (Pin_3)
- net DISTANCE_L_OUT: now also J7.4 (Pin_4)
- net DISTANCE_R90_OUT: now also J2.3 (Pin_3)
- net DISTANCE_R_OUT: now also J2.4 (Pin_4)
- net GND: now also J2.1 (Pin_1), J7.1 (Pin_1), J8.1 (Pin_1)
- net LINE_LEFT_OUT: now also J7.6 (Pin_6)
- net LINE_RIGHT_OUT: now also J2.6 (Pin_6)
- net DISTANCE_LF: no longer names the net of U5.7 (A6)
- net DISTANCE_LF_OUT: no longer names the net of U5.14 (B6)
- net DISTANCE_RF renamed DISTANCE_CENTER
- net DISTANCE_RF_OUT renamed DISTANCE_CENTER_OUT
- net DISTANCE_CENTER_OUT: now also J2.5 (Pin_5)
- new net SERVO: J8.3 (Pin_3)
- no-connect marks 4 -> 7
Other:
- moved on the sheet: R21, R22, R23, R24
